File: pcb-devboard/pcb-devboard.kicad_sch (KiCad schematic)
At the start: 24 parts

Commit message: Schematic improvements and first layout draft
Parts:
- removed R? (x2): 4.7k, Resistor_SMD:R_0402_1005Metric, symbol Device:R_US
- added R6, R7, R8: 5.1K 0402, Resistor_SMD:R_0402_1005Metric, symbol Device:R_Small
- added TP1: TestPoint, mine:TestPoint_Pad_1.0x1.0mm, symbol Connector:TestPoint
- D1: renamed from D?; footprint LED_THT:LED_D5.0mm -> LED_SMD:LED_0603_1608Metric; LCSC (none) -> C2286
- JP1, JP2, JP3, JP4, JP5: renamed from JP?; footprint (none) -> Jumper:SolderJumper-2_P1.3mm_Open_Pad1.0x1.5mm
- gave numbers to parts that had none: 16
Connections:
- net GND: now also R4.2; no longer R5.2
- net PIN_PA0: now also R8.2
- net VBUS: now also R5.1; no longer R4.1
- net VBUS_SENSE: now also R4.1, R5.2, TP1.1; no longer R4.2, R5.1
- net at J1.2 (Pin_2): now also R8.1
- net at U1.6 (TNOW): now also R6.1, R7.2
- net at D1.2 (A): now also R6.2, R7.1
Other:
- moved on the sheet: C4, D1, J1, J2, J3, JP1, JP2, JP3, JP4, JP5, R4, R5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
