File: pcb-devboard/pcb-devboard.kicad_pcb (KiCad board)
At the start: 2 copper layers, 11.4 x 44.3 mm, 26 parts, among them J1 UPDI_PROGRAMMER, J2 PINS1, J3 PINS2, U1 CH340E, U2 ATtiny412-SS

Commit message: Layout improvements
Parts:
- J1: moved to B.Cu
- R8: moved to F.Cu
- moved J2 7.62 mm to (142.2, 119.4)
- moved J3 7.62 mm to (149.9, 119.4)
- moved R8 3.08 mm to (146.9, 109.4), turned to 180 degrees
- moved TP1 0.20 mm to (141.5, 97.2)
- turned J1 to 180 degrees
Routing:
- net /VBUS: track 4.17 -> 11.1 mm
- net /PIN_PA0: track 11.4 -> 18.0 mm, vias 1 -> 0
- net /PIN_PA1: track 26.3 -> 20.8 mm, vias 3 -> 2
- net GND: track 0.00 -> 5.31 mm, vias 0 -> 6
- net VSYS: track 40.2 -> 37.3 mm, vias 4 -> 5
- net /PIN_PA7: track 20.0 -> 22.8 mm, vias 3 -> 4
- net /PIN_PA6: track 21.5 -> 23.6 mm, vias 1 -> 2
- net /PIN_PA3: track 16.8 -> 18.7 mm, vias 1 -> 2
- net Net-(J1-Pad2): track 1.70 -> 3.27 mm
- net /PIN_PA2: track 26.6 -> 26.5 mm, vias 0 -> 2
Other:
- board text added: "0"
- board text added: "1"
- board text added: "2"
- board text added: "3"
- board text added: "6"
- board text added: "7"
- board text added: "A"
- board text added: "D"
- board text added: "PORT A"
- board text added: "PPWR"
