File: pcb-interface/pcb-interface.kicad_pcb (KiCad board)
At the start: 2 copper layers, 52.1 x 49.9 mm, 28 parts, among them J1 UPDI_PROGRAMMER, J2 PINS1, J3 PINS2, J4 PINS1, J5 PINS1, U1 CH340E, U2 ATtiny412-SS

Commit message: 41x interface board: Version 1.0 as manufactured
Parts:
- removed C3: 0.1μF, Capacitor_SMD:C_0603_1608Metric
- removed J2: PINS1, Connector_PinHeader_2.54mm:PinHeader_1x10_P2.54mm_Vertical
- removed J3: PINS2, Connector_PinHeader_2.54mm:PinHeader_1x10_P2.54mm_Vertical
- removed J4: PINS1, Connector_PinHeader_2.54mm:PinHeader_2x04_P2.54mm_Vertical
- removed U2: ATtiny412-SS, Package_SO:SOIC-20W_7.5x12.8mm_P1.27mm
- moved R8 6.09 mm to (73.7, 95.1)
- moved J1 3.76 mm to (71.1, 97.7), turned to 90 degrees
- moved C1 3.25 mm to (70.8, 112.2)
- moved R1 3.25 mm to (73.3, 112.9)
- moved R3 3.25 mm to (79.4, 112.4)
- moved R4 3.25 mm to (78.0, 110.8)
- moved C2 3.25 mm to (72.7, 108.5)
- moved C4 3.25 mm to (70.8, 109.0)
- moved D1 3.25 mm to (79.6, 105.3)
- moved JP1 3.25 mm to (71.2, 104.9)
- moved JP2 3.25 mm to (76.6, 101.9)
- moved JP3 3.25 mm to (73.9, 101.9)
- moved JP4 3.25 mm to (79.2, 101.9)
- moved JP5 3.25 mm to (71.2, 101.9)
- moved NT1 3.25 mm to (72.2, 112.4)
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Routing:
- net /PIN_PA7: track 61.2 -> 9.48 mm, vias 3 -> 1
- net /PIN_PA6: track 66.1 -> 15.7 mm, vias 4 -> 2
- net /PIN_PA2: track 59.7 -> 17.8 mm, vias 4 -> 2
- net /PIN_PC3: track 40.6 -> 0.00 mm, vias 2 -> 0
- net /PIN_PC2: track 37.2 -> 0.00 mm, vias 2 -> 0
- net /PIN_PA5: track 36.2 -> 0.00 mm, vias 2 -> 0
- net /PIN_PA0: track 42.0 -> 6.03 mm
- net /PIN_PA4: track 35.8 -> 0.00 mm, vias 2 -> 0
- net /PIN_PA1: track 46.4 -> 11.7 mm, vias 3 -> 1
- net /PIN_PA3: track 34.6 -> 0.00 mm, vias 2 -> 0
- net /PIN_PC1: track 33.8 -> 0.00 mm, vias 2 -> 0
- net VSYS: track 60.6 -> 29.5 mm, vias 6 -> 3
- net /PIN_PC0: track 30.1 -> 0.00 mm, vias 2 -> 0
- net /PIN_PB0: track 28.3 -> 0.00 mm, vias 1 -> 0
- net /PIN_PB5: track 25.5 -> 0.00 mm
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Other:
- board size 52.1 x 49.9 mm -> 11.9 x 34.7 mm
- board text added: "5V"
- board text added: "USB-C"
- board text added: "by Tarn"
- board text removed: "0"
- board text removed: "1"
- board text removed: "2"
- board text removed: "3"
- board text removed: "6"
- board text removed: "7"
- board text removed: "PORT A"
