File: pcb-interface/pcb-interface.kicad_sch (KiCad schematic)
At the start: 28 parts, among them J1 UPDI_PROGRAMMER, J2 PINS1, J3 PINS2, J4 PINS1, J5 PINS1, U1 CH340E, U2 ATtiny412-SS

Commit message: 41x interface board: Version 1.0 as manufactured
Parts:
- removed C3: 0.1μF, Capacitor_SMD:C_0603_1608Metric, symbol Device:C
- removed J2: PINS1, Connector_PinHeader_2.54mm:PinHeader_1x10_P2.54mm_Vertical, symbol Connector:Conn_01x10_Male
- removed J3: PINS2, Connector_PinHeader_2.54mm:PinHeader_1x10_P2.54mm_Vertical, symbol Connector:Conn_01x10_Male
- removed J4: PINS1, Connector_PinHeader_2.54mm:PinHeader_2x04_P2.54mm_Vertical, symbol Connector_Generic:Conn_02x04_Odd_Even
- removed U2: ATtiny412-SS, Package_SO:SOIC-20W_7.5x12.8mm_P1.27mm, symbol MCU_Microchip_ATtiny:ATtiny416-S
- R1, R2, R6, R7, R8: LCSC C25941 -> C25905
- R5: LCSC C2906885 -> C25744
Connections:
- no-connect marks 5 -> 4
Other:
- note removed: "REPLACE WITH 0805!"
